Commit message: Added gui.

File: ihe_hardware/turtlebot_xtion_top_description/urdf/xtion.xacro (robot description, xacro)
@@ -1,4 +1,5 @@
 <?xml version="1.0"?>
 <robot name="xtion" xmlns:xacro="http://ros.org/wiki/xacro">
+  <include filename="$(find turtlebot_description)/urdf/turtlebot_hardware.urdf.xacro" />
   <property name="M_PI" value="3.14159" />
   <xacro:macro name="xtion" params="parent x_loc y_loc z_loc rr rp ry">
@@ -30,6 +31,5 @@
     <!-- platform for xtion -->
     <joint name="base_xtion_platform_joint" type="fixed">
-      <origin xyz="${x_loc} ${y_loc} ${z_loc}"
-              rpy="${rr} ${rp} ${ry}" />
+      <origin xyz="${x_loc} ${y_loc} ${z_loc}" rpy="${rr} ${rp} ${ry}" />
       <parent link="${parent}" />
       <child link="xtion_platform" />

Commit message: Added xtion45 clips. Minor changes to GUI.

File: ihe_hardware/turtlebot_xtion_top_description/urdf/xtion.xacro (robot description, xacro)
@@ -1,5 +1,4 @@
 <?xml version="1.0"?>
 <robot name="xtion" xmlns:xacro="http://ros.org/wiki/xacro">
-  <include filename="$(find turtlebot_description)/urdf/turtlebot_hardware.urdf.xacro" />
   <property name="M_PI" value="3.14159" />
   <xacro:macro name="xtion" params="parent x_loc y_loc z_loc rr rp ry">
@@ -151,3 +150,48 @@
     </link>
   </xacro:macro>
+  <!-- xtion 45 clips -->
+  <xacro:macro name="xtion45_left_clip"
+               params="parent number x_loc y_loc z_loc">
+    <joint name="xtion45_left_clip_${number}_joint" type="fixed">
+      <origin xyz="${x_loc} ${y_loc} ${z_loc}"
+              rpy="${M_PI/2} 0 0" />
+      <parent link="${parent}" />
+      <child link="xtion45_left_clip_${number}_link" />
+    </joint>
+    <link name="xtion45_left_clip_${number}_link">
+      <inertial>
+        <mass value="0.01" />
+        <origin xyz="0 0 0" />
+        <inertia ixx="0.001" ixy="0" ixz="0" iyy="0.001" iyz="0" izz="0.001" />
+      </inertial>
+      <visual>
+        <origin xyz="0 0 0" rpy="0 0 0" />
+        <geometry>
+          <mesh filename="package://turtlebot_xtion_top_description/meshes/xtion/xtion45_clip_left.dae" scale="0.001 0.001 0.001" />
+        </geometry>
+      </visual>
+    </link>
+  </xacro:macro>
+  <xacro:macro name="xtion45_right_clip"
+               params="parent number x_loc y_loc z_loc">
+    <joint name="xtion45_right_clip_${number}_joint" type="fixed">
+      <origin xyz="${x_loc} ${y_loc} ${z_loc}"
+              rpy="${-M_PI/2} 0 0" />
+      <parent link="${parent}" />
+      <child link="xtion45_right_clip_${number}_link" />
+    </joint>
+    <link name="xtion45_right_clip_${number}_link">
+      <inertial>
+        <mass value="0.01" />
+        <origin xyz="0 0 0" />
+        <inertia ixx="0.001" ixy="0" ixz="0" iyy="0.001" iyz="0" izz="0.001" />
+      </inertial>
+      <visual>
+        <origin xyz="0 0 0" rpy="0 0 0" />
+        <geometry>
+          <mesh filename="package://turtlebot_xtion_top_description/meshes/xtion/xtion45_clip_right.dae" scale="0.001 0.001 0.001" />
+        </geometry>
+      </visual>
+    </link>
+  </xacro:macro>
 </robot>

File: ihe_hardware/urdf_compose/urdf/kinect.xacro (robot description, xacro)
@@ -3,5 +3,4 @@
   <property name="M_PI" value="3.14159"/>
   <include filename="$(find turtlebot_description)/urdf/gazebo.urdf.xacro"/>
-  <include filename="$(find turtlebot_description)/urdf/turtlebot_hardware.urdf.xacro"/>
 <xacro:macro name="turtlebot_kinect"
              params="parent cam_x cam_y cam_z cam_rr cam_rp cam_ry">
