Commit message: Added urdf for Xtended Xtion mount.

File: ihe_hardware/turtlebot_xtion_top_description/urdf/turtlebot.xacro (robot description, xacro)
@@ -411,5 +411,5 @@
       <origin xyz="0.0 0.0 0.0" rpy="0 0 0" />
       <geometry>
-        <box size="0.05 0.24 0.02"/>
+        <box size="0.05 0.246 0.02"/>
       </geometry>
     </collision>

File: ihe_hardware/turtlebot_xtion_top_description/urdf/xtion.xacro (robot description, xacro)
@@ -50,5 +50,5 @@
         <origin xyz="0.0 0.0 0.0" rpy="0 0 0" />
         <geometry>
-          <box size="0.05 0.24 0.02"/>
+          <box size="0.05 0.246 0.02"/>
         </geometry>
       </collision>
@@ -155,5 +155,5 @@
     <joint name="xtion45_left_clip_${number}_joint" type="fixed">
       <origin xyz="${x_loc} ${y_loc} ${z_loc}"
-              rpy="${M_PI/2} 0 0" />
+              rpy="0 0 0" />
       <parent link="${parent}" />
       <child link="xtion45_left_clip_${number}_link" />
@@ -177,5 +177,5 @@
     <joint name="xtion45_right_clip_${number}_joint" type="fixed">
       <origin xyz="${x_loc} ${y_loc} ${z_loc}"
-              rpy="${-M_PI/2} 0 0" />
+              rpy="0 0 0" />
       <parent link="${parent}" />
       <child link="xtion45_right_clip_${number}_link" />
@@ -195,3 +195,30 @@
     </link>
   </xacro:macro>
+  <!-- extension plate -->
+  <xacro:macro name="plate_xtension" params="parent x_loc y_loc z_loc">
+    <joint name="plate_xtension_joint" type="fixed">
+      <origin xyz="${x_loc} ${y_loc} ${z_loc}" rpy="0 0 0" />
+      <parent link="${parent}" />
+      <child link="plate_xtension_link" />
+    </joint>
+    <link name="plate_xtension_link">
+      <inertial>
+        <mass value="0.01" />
+        <origin xyz="0 0 0" />
+        <inertia ixx="0.001" ixy="0" ixz="0" iyy="0.001" iyz="0" izz="0.001" />
+      </inertial>
+      <visual>
+        <origin xyz="0 0 0" rpy="0 0 0" />
+        <geometry>
+          <mesh filename="package://turtlebot_xtion_top_description/meshes/xtion/xtend_plate.dae" scale="0.001 0.001 0.001" />
+        </geometry>
+      </visual>
+      <collision>
+        <origin xyz="0.0265 0.0 0.0032005" rpy="0 0 0" />
+        <geometry>
+          <box size="0.066 0.28 0.006401"/>
+        </geometry>
+      </collision>
+    </link>
+  </xacro:macro>
 </robot>
