Commit message: Adding urdf for TurtleBot Metric Version.

File: ihe_hardware/turtlebot_body/urdf/turtlebot_metric.xacro (robot description, xacro)
@@ -13,13 +13,4 @@
   <!-- base_footprint is a fictitious link(frame) that is on the ground right below base_link origin, navigation stack depends on this frame -->
   <link name="base_footprint">
-<!--
-    <inertial>
-      <mass value="0.0001" />
-      <origin xyz="0 0 0" />
-      <inertia ixx="0.0001" ixy="0.0" ixz="0.0"
-              iyy="0.0001" iyz="0.0"
-              izz="0.0001" />
-    </inertial>
--->
     <visual>
       <origin xyz="0 0 0" rpy="0 0 0" />
@@ -283,7 +274,7 @@
     </inertial>
     <visual>
-      <origin xyz=" 0 0 0 " rpy="0 0 0" />
-      <geometry>
-        <mesh filename="package://turtlebot_description/meshes/plate_0_logo.dae"/>
+      <origin xyz="0 0 0 " rpy="0 0 0" />
+      <geometry>
+        <mesh filename="package://turtlebot_body/meshes/disk_00_hex.dae" scale="0.001 0.001 0.001"/>
       </geometry>
     </visual>
@@ -300,5 +291,5 @@
   <turtlebot_standoff_2in parent="base_link" number="3" x_loc="-0.052832" y_loc="0.1314196" z_loc="0.0709803"/>
   <joint name="plate_1_joint" type="fixed">
-    <origin xyz="0.04068 0 0.05715" rpy="0 0 0" />
+    <origin xyz="0.04068 0 0.054" rpy="0 0 0" />
     <parent link="plate_0_link"/>
     <child link="plate_1_link" />
@@ -313,7 +304,7 @@
     </inertial>
     <visual>
-      <origin xyz=" 0 0 0 " rpy="0 0 0" />
-      <geometry>
-        <mesh filename="package://turtlebot_description/meshes/plate_1_logo.dae"/>
+      <origin xyz="0 0 0 " rpy="${M_PI/2} 0 ${M_PI/2}" />
+      <geometry>
+        <mesh filename="package://turtlebot_body/meshes/disk_01_hex.dae" scale="0.001 0.001 0.001"/>
       </geometry>
     </visual>
@@ -343,7 +334,7 @@
     </inertial>
     <visual>
-      <origin xyz=" 0 0 0 " rpy="0 0 0" />
-      <geometry>
-        <mesh filename="package://turtlebot_description/meshes/plate_1_logo.dae"/>
+      <origin xyz="0 0 0 " rpy="${M_PI/2} 0 ${M_PI/2}" />
+      <geometry>
+        <mesh filename="package://turtlebot_body/meshes/disk_02_hex.dae" scale="0.001 0.001 0.001"/>
       </geometry>
     </visual>
@@ -360,5 +351,5 @@
   <turtlebot_standoff_8in parent="standoff_2in_7_link" number="3" x_loc="0" y_loc="0" z_loc="0.05715"/>
   <joint name="plate_3_joint" type="fixed">
-    <origin xyz="-0.01316 0 0.2063496" rpy="0 0 0" />
+    <origin xyz="0 0 0.2094996" rpy="0 0 0" />
     <parent link="plate_2_link"/>
     <child link="plate_3_link" />
@@ -373,7 +364,7 @@
     </inertial>
     <visual>
-      <origin xyz=" 0 0 0 " rpy="0 0 0" />
-      <geometry>
-        <mesh filename="package://turtlebot_description/meshes/plate_2_logo.dae"/>
+      <origin xyz="0 0 0" rpy="${M_PI/2} 0 ${M_PI/2}" />
+      <geometry>
+        <mesh filename="package://turtlebot_body/meshes/disk_03_hex.dae" scale="0.001 0.001 0.001"/>
       </geometry>
     </visual>

File: ihe_hardware/turtlebot_xtion_top_description/urdf/xtion.xacro (robot description, xacro)
@@ -56,5 +56,5 @@
     <!-- left clip for xtion -->
     <joint name="base_xtion_left_clip_joint" type="fixed">
-      <origin xyz="0.017 -0.0745 0.00635"
+      <origin xyz="-0.017 -0.0745 0.00635"
               rpy="0.0 0.0 0.0" />
       <parent link="xtion_platform" />
