Commit message: Minor changes to urdfs.

File: ihe_hardware/turtlebot_body/urdf/turtlebot_metric.urdf.xacro (robot description, xacro)
@@ -3,3 +3,8 @@
   <include filename="$(find turtlebot_body)/urdf/turtlebot_metric.xacro"/>
   <turtlebot_body/>
+  <include filename="$(find urdf_compose)/urdf/kinect.xacro"/>
+  <include filename="$(find turtlebot_xtion_top_description)/urdf/turtlebot_hardware.xacro"/>
+  <turtlebot_standoff_kinect number="0" parent="plate_2_link" x_loc="-0.102438" y_loc="-0.098" z_loc="0.003201"/>
+  <turtlebot_standoff_kinect number="1" parent="plate_2_link" x_loc="-0.102438" y_loc="0.098" z_loc="0.003201"/>
+  <turtlebot_kinect cam_rp="0" cam_rr="0" cam_ry="0" cam_x="-0.0844382" cam_y="0" cam_z="0.10475" parent="plate_2_link"/>
 </robot>

File: ihe_hardware/turtlebot_xtion_top_description/urdf/turtlebot.xacro (robot description, xacro)
@@ -417,5 +417,5 @@
   <!-- left clip for xtion -->
   <joint name="base_xtion_left_clip_joint" type="fixed">
-    <origin xyz="0.017 -0.0745 0.00635"
+    <origin xyz="-0.017 -0.0745 0.00635"
             rpy="0.0 0.0 0.0" />
     <parent link="xtion_platform" />
