Commit message: Renaming package to turtlebot_metric_description.

File: ihe_hardware/turtlebot_metric_description/urdf/turtlebot_metric.urdf.xacro (robot description, xacro)
@@ -1,5 +1,5 @@
 <?xml version="1.0" ?>
 <robot name="turtlebot" xmlns:controller="http://playerstage.sourceforge.net/gazebo/xmlschema/#controller" xmlns:interface="http://playerstage.sourceforge.net/gazebo/xmlschema/#interface" xmlns:sensor="http://playerstage.sourceforge.net/gazebo/xmlschema/#sensor" xmlns:xacro="http://ros.org/wiki/xacro">
-  <include filename="$(find turtlebot_body)/urdf/turtlebot_metric.xacro"/>
+  <include filename="$(find turtlebot_metric_description)/urdf/turtlebot_metric.xacro"/>
   <turtlebot_body/>
   <include filename="$(find urdf_compose)/urdf/kinect.xacro"/>

File: ihe_hardware/turtlebot_metric_description/urdf/turtlebot_metric.xacro (robot description, xacro)
@@ -276,5 +276,5 @@
       <origin xyz="0 0 0 " rpy="0 0 0" />
       <geometry>
-        <mesh filename="package://turtlebot_body/meshes/disk_00_hex.dae" scale="0.001 0.001 0.001"/>
+        <mesh filename="package://turtlebot_metric_description/meshes/disk_00_hex.dae" scale="0.001 0.001 0.001"/>
       </geometry>
     </visual>
@@ -306,5 +306,5 @@
       <origin xyz="0 0 0 " rpy="${M_PI/2} 0 ${M_PI/2}" />
       <geometry>
-        <mesh filename="package://turtlebot_body/meshes/disk_01_hex.dae" scale="0.001 0.001 0.001"/>
+        <mesh filename="package://turtlebot_metric_description/meshes/disk_01_hex.dae" scale="0.001 0.001 0.001"/>
       </geometry>
     </visual>
@@ -336,5 +336,5 @@
       <origin xyz="0 0 0 " rpy="${M_PI/2} 0 ${M_PI/2}" />
       <geometry>
-        <mesh filename="package://turtlebot_body/meshes/disk_02_hex.dae" scale="0.001 0.001 0.001"/>
+        <mesh filename="package://turtlebot_metric_description/meshes/disk_02_hex.dae" scale="0.001 0.001 0.001"/>
       </geometry>
     </visual>
@@ -366,5 +366,5 @@
       <origin xyz="0 0 0" rpy="${M_PI/2} 0 ${M_PI/2}" />
       <geometry>
-        <mesh filename="package://turtlebot_body/meshes/disk_03_hex.dae" scale="0.001 0.001 0.001"/>
+        <mesh filename="package://turtlebot_metric_description/meshes/disk_03_hex.dae" scale="0.001 0.001 0.001"/>
       </geometry>
     </visual>
